Commit message: Update files

File: mkmr_sw_urdf/urdf/mkmr_urdf.urdf (robot description, URDF)
Before this commit: robot mkmr_urdf, 13 links, 12 joints
Links:
- link back_left_wheel: mass 0.0560724795860692 -> 0.0476113796200164
- link back_right_wheel: mass 0.0560727186165722 -> 0.0476116186505194
- link base_link: mass 0.10356 -> 0.103562496069832
- link camera: mass 0.0025101 -> 0.0025100794824479
- link chasis_link: mass 0.00099699 -> 0.00099698897376
- link fBattery: mass 1 -> 0.97961835817872
- link fDrivers: mass 0.038483 -> 0.0384827950773915
- link fMotor: mass 0.178561366362791 -> 0.212405766227002
- link fMotorBracket: mass 0.012335 -> 0.012334653543211
- link fPC: mass 1 -> 0.8130163223512
- link front_left_wheel: mass 0.0560727186165723 -> 0.0476116186505196
- link front_right_wheel: mass 0.0560724795860693 -> 0.0476113796200165
- link scan: mass 1.3308 -> 1.33076913637071
Joints:
- joint back_left_wheel_joint: origin xyz=-0.082516 0.079 0 rpy=-3.1416 0 -1.5708 -> xyz=-0.0825159999999995 0.0924999999999993 0 rpy=-3.14159265358979 0 0
- joint back_right_wheel_joint: origin xyz=-0.082516 -0.079 0 rpy=-3.1416 0 -1.5708 -> xyz=-0.0825159999999981 -0.0945000000000007 0 rpy=-3.14159265358979 0 0
- joint camera_joint: origin xyz=0.08282 -0.07342 -0.036649 rpy=1.5708 1.5708 0 -> xyz=0.08282 -0.0734200000000002 -0.036649 rpy=1.5707963267949 1.5707963267949 0
- joint chasis_joint: origin xyz=-0.032984 0.0355 0 rpy=1.5708 0 0 -> xyz=-0.032984000000001 0.0355 0 rpy=1.5707963267949 0 0
- joint fBattery_joint: origin xyz=-0.09476 -0.047958 0 rpy=-3.1416 0 0 -> xyz=-0.09476040070881 -0.047958 0 rpy=-3.14159265358979 0 0
- joint fDrivers_joint: origin xyz=-0.039948 0.004651 0.037727 rpy=-1.5708 0 -3.1416 -> xyz=-0.0399479 0.00465100000000018 0.037726592766333 rpy=-1.5707963267949 0 -3.14159265358979
- joint fMotorBracket_joint: origin xyz=0 0 0 rpy=1.5708 1.5708 0 -> xyz=0.0345000000000004 0 -0.0609999999999998 rpy=1.5707963267949 1.5707963267949 0
- joint fMotor_joint: origin xyz=0 0 0 rpy=0 0 0 -> xyz=0.0179999999999999 -0.15 -0.0285000000000011 rpy=0 1.5707963267949 0
- joint fPC_joint: origin xyz=0.02413 -0.03221 0 rpy=3.1416 1.5708 0 -> xyz=0.02413 -0.0322100000000002 0 rpy=3.14159265358979 1.5707963267949 0
- joint front_left_wheel_joint: origin xyz=0.082484 0.079 0 rpy=3.1416 0 1.5708 -> xyz=0.0824840000000006 0.0945000000000005 0 rpy=3.14159265358979 0 -3.14159265358979
- joint front_right_wheel_joint: origin xyz=0.082484 -0.079 0 rpy=3.1416 0 1.5708 -> xyz=0.0824840000000019 -0.0924999999999995 0 rpy=3.14159265358979 0 -3.14159265358979
- joint scan_joint: origin xyz=0.054864 -0.08602 -0.000762 rpy=3.1416 1.5708 0 -> xyz=0.054864 -0.0860200000000002 -0.000761999999999532 rpy=3.14159265358979 1.5707963267949 0
